File: wv_battery_interface.kicad_pcb (KiCad board)
At the start: 2 copper layers, 60.5 x 54 mm, 36 parts, among them J1 Conn_01x03, J10 Conn_01x05, J11 Conn_01x03, J2 Conn_01x03, J3 Conn_01x04, J4 Conn_01x03, J5 Conn_01x02, J6 Conn_01x03, J7 Conn_01x02, J8 Conn_01x04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

Commit message: alternate component values added
Parts:
- Q1, Q3: value SI01P10 -> P-channel MOSFET, 100V@1A
- R3, R6: value 1kΩ -> 100kΩ
Connections:
- net /Soft Latch Switch 1/Switch-GND renamed /Soft Latch Switch 1/Switch-to-GND
- D2 pad : (no net) -> +BATT1
- D4 pad : (no net) -> +BATT2
